Commit message: Add hand hardware profiles and launch wrappers

File: ros2_control/silverhand_hand.ros2_control.xacro (robot description, xacro)
@@ -3,5 +3,5 @@
   <xacro:macro
     name="silverhand_hand_ros2_control"
-    params="name initial_positions_file use_mock_hardware:=true can_iface:=can0 node_id:=120">
+    params="name initial_positions_file prefix:='' use_mock_hardware:=true can_iface:=can0 node_id:=120 queue_len:=1000">
     <xacro:property
       name="initial_positions"
@@ -19,7 +19,8 @@
           <param name="can_iface">${can_iface}</param>
           <param name="node_id">${node_id}</param>
+          <param name="queue_len">${queue_len}</param>
         </xacro:unless>
       </hardware>
-      <joint name="left_finger_joint">
+      <joint name="${prefix}left_finger_joint">
         <command_interface name="position"/>
         <command_interface name="effort"/>
@@ -30,5 +31,5 @@
         <state_interface name="effort"/>
       </joint>
-      <joint name="right_finger_joint">
+      <joint name="${prefix}right_finger_joint">
         <command_interface name="position"/>
         <command_interface name="effort"/>

File: urdf/silverhand_hand.urdf.xacro (robot description, xacro)
@@ -9,4 +9,5 @@
   <xacro:arg name="can_iface" default="can0"/>
   <xacro:arg name="node_id" default="120"/>
+  <xacro:arg name="queue_len" default="1000"/>
   <xacro:silverhand_hand_ros2_control
     name="SilverhandHandSystem"
@@ -14,4 +15,5 @@
     use_mock_hardware="$(arg use_mock_hardware)"
     can_iface="$(arg can_iface)"
-    node_id="$(arg node_id)"/>
+    node_id="$(arg node_id)"
+    queue_len="$(arg queue_len)"/>
 </robot>
